File: pcb_challenge_final.kicad_pcb (KiCad board)
At the start: 4 copper layers, 39.5 x 39.5 mm, 164 parts, among them J4 Conn_01x04_Pin, J5 Conn_01x04_Pin, Q15 Q_Dual_NPN_PNP_B1E2B2C2E1C1, Q16 Q_Dual_NPN_PNP_B1E2B2C2E1C1, Q17 Q_Dual_NPN_PNP_B1E2B2C2E1C1, Q18 Q_Dual_NPN_PNP_B1E2B2C2E1C1, Q19 Q_Dual_NPN_PNP_B1E2B2C2E1C1, Q20 Q_Dual_NPN_PNP_B1E2B2C2E1C1, Q21 Q_Dual_NPN_PNP_B1E2B2C2E1C1, Q22 Q_Dual_NPN_PNP_B1E2B2C2E1C1, Q23 Q_Dual_NPN_PNP_B1E2B2C2E1C1, Q24 Q_Dual_NPN_PNP_B1E2B2C2E1C1, Q25 Q_Dual_NPN_PNP_B1E2B2C2E1C1, Q26 Q_Dual_NPN_PNP_B1E2B2C2E1C1, Q27 Q_Dual_NPN_PNP_B1E2B2C2E1C1, Q28 Q_Dual_NPN_PNP_B1E2B2C2E1C1, Q29 Q_Dual_NPN_PNP_B1E2B2C2E1C1, SW1 SW_Push, SW2 SW_Push, SW3 SW_Push, U1 74AUP1G80, U10 NMUX1308BQ, U11 NMUX1308BQ, U12 NMUX1308BQ, U13 NMUX1308BQ, U14 NMUX1308BQ, U15 NMUX1308BQ, U16 NMUX1308BQ, U17 74AUP1G80, U18 74AHC1G86, U19 74AUP1G80, U20 74AUP1G80, U21 74LV1T08GV, U22 CD74HC283M96, U23 74LV1T08GV, U24 74LVC1GU04DRL, U25 ESP32-S3-MINI-1, U26 74LVC1GU04DRL, U27 74LV1T08GV, U28 CD74HC283M96, U29 NMUX1308BQ, U3 74AHC1G86, U30 NMUX1308BQ, U31 NMUX1308BQ, U32 NMUX1308BQ, U33 74AUP1G80, U34 74AUP1G80, U35 NMUX1308BQ, U36 NMUX1308BQ, U37 74AUP1G80, U38 74AUP1G80, U39 NMUX1308BQ, U4 74AUP1G80, U40 NMUX1308BQ, U41 NMUX1308BQ, U42 NMUX1308BQ, U43 NMUX1308BQ, U44 NMUX1308BQ, U45 74AUP1G80, U46 74AUP1G80, U47 74AUP1G80, U48 74AUP1G80, U49 74AUP1G80, U5 74AUP1G80, U50 74AUP1G80, U51 74LV1T08GV, U52 74AHC1G86, U53 74LVC1GU04DRL, U54 74LVC1GU04DRL, U55 74AHC1G86, U56 74AHC1G86, U57 74LVC1GU04DRL, U58 74LVC1GU04DRL, U59 74LV1T08GV, U6 74AUP1G80, U60 74AHC1G86, U61 74LVC1GU04DRL, U62 74LV1T08GV, U63 74LV1T08GV, U64 NMUX1308BQ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

Commit message: Add files via upload
Parts:
- moved U22 1.78 mm to (51.1, 58.9)
Routing:
- net rst: track 0.00 -> 83.8 mm, vias 0 -> 2
- net IO8: track 0.00 -> 82.9 mm, vias 0 -> 3
- net +3.3V: track 0.00 -> 82.1 mm, vias 0 -> 2
- net ???: track 0.00 -> 67.3 mm, vias 0 -> 2
- net Net-(U25-GND-Pad2): track 0.00 -> 66.9 mm, vias 0 -> 2
- net GND: track 0.00 -> 63.1 mm, vias 0 -> 14
- net USB_D+: track 0.00 -> 55.0 mm, vias 0 -> 3
- net rc1: track 0.00 -> 51.5 mm, vias 0 -> 4
- net Net-(Q26A-C1): track 0.00 -> 51.0 mm, vias 0 -> 3
- net Net-(U22-CIN): track 0.00 -> 50.3 mm, vias 0 -> 2
- net Net-(U59-B): track 0.00 -> 47.4 mm, vias 0 -> 2
- net Net-(U25-IO15): track 0.00 -> 46.3 mm, vias 0 -> 3
- net r_en: track 0.00 -> 45.2 mm, vias 0 -> 4
- net Net-(U63-Y): track 0.00 -> 44.4 mm, vias 0 -> 2
- net EN: track 0.00 -> 43.9 mm
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